Commit message: [feat] add new STL files and update URDF for probe base and end effector integration

File: xarm_description/urdf/lite6/lite6.urdf.xacro (robot description, xacro)
@@ -208,10 +208,47 @@
       <dynamics damping="1.0" friction="1.0"/>
     </joint>
-    <!-- <link name="${prefix}link_eef" />
-    <joint name="${prefix}joint_eef" type="fixed">
-      <origin xyz="0 0 0" rpy="0 0 0" />
+    <link name="${prefix}link_end" />
+    <joint name="${prefix}joint_end" type="fixed">
+      <origin xyz="0 0 0" rpy="${pi} 0 ${pi/2}" />
       <parent link="${prefix}link6" />
-      <child link="${prefix}link_eef" />
-    </joint> -->
+      <child link="${prefix}link_end" />
+    </joint>
+    <!-- force sensor urdf -->
+    <xacro:include filename="$(find rokubimini_description)/urdf/BFT_SENS_ECAT_M8.urdf.xacro" />
+    <xacro:BFT_SENS_ECAT_M8 prefix="ft_sensor0" />
+    <joint name="bota_ft_sensor" type="fixed">
+    <parent link="${prefix}link_end"/>
+    <child link = "ft_sensor0_mounting" />
+    <origin xyz="0.0 0.0 0.0" rpy="${pi} 0.0 ${pi/2}" />
+    </joint>
+    <link name="probe_base">
+    <inertial>
+      <origin rpy="0 0 0" xyz="0 0 0"/>
+       <mass value="0.0"/>
+       <inertia ixx="0" ixy="0" ixz="0" iyy="0" iyz="0" izz="0"/>
+    </inertial>
+    <xacro:common_link_visual
+        mesh_filename="lite6/visual/punta_robot"
+        origin_xyz="0 0 0.01"
+        origin_rpy="0 0 0"
+        material_name="${prefix}Silver" />
+    <xacro:common_link_collision
+        mesh_filename="lite6/collision/punta_robot"
+        origin_xyz="0 0 0.01"
+        origin_rpy="0 0 0" />
+    </link>
+    <joint name="base_tool" type="fixed">
+    <parent link="ft_sensor0_wrench" />
+    <child link = "probe_base" />
+    <origin xyz="0.0 0.0 0.0" rpy="0.0 0.0 0.0" />
+    </joint>
+    <link
+      name="probe">
+    </link>
+    <joint name="tip_tool" type="fixed">
+    <parent link="ft_sensor0_wrench" />
+    <child link = "probe" />
+    <origin xyz="0.0 0.0 0.0625" rpy="0.0 0.0 0.0" />
+    </joint>
   </xacro:macro>
 </robot>

File: xarm_description/urdf/xarm_device.urdf.xacro (robot description, xacro)
@@ -11,5 +11,5 @@
   <xacro:arg name="model1300" default="false"/>
   <xacro:arg name="dof" default="7"/>
-  <xacro:arg name="robot_ip" default=""/>
+  <xacro:arg name="robot_ip" default="192.168.1.164"/>
   <xacro:arg name="robot_type" default="xarm"/>
   <xacro:arg name="robot_sn" default=""/>

Commit message: Added mounting and RS to the urdf

File: xarm_description/urdf/lite6/lite6.urdf.xacro (robot description, xacro)
@@ -210,5 +210,5 @@
     <link name="${prefix}link_end" />
     <joint name="${prefix}joint_end" type="fixed">
-      <origin xyz="0 0 0" rpy="${pi} 0 ${pi/2}" />
+      <origin xyz="0 0 0.003" rpy="${pi} 0 ${pi/2}" />
       <parent link="${prefix}link6" />
       <child link="${prefix}link_end" />
@@ -251,4 +251,36 @@
     <origin xyz="0.0 0.0 0.0625" rpy="0.0 0.0 0.0" />
     </joint>
+    <joint name="camera_mounting" type="fixed">
+    <parent link="ft_sensor0_mech3"/>
+    <child link = "mounting" />
+      <origin xyz="0.0 0.0 0.0" rpy="0.0 0.0 ${pi/2}"/>
+    </joint>
+    <link name="mounting">
+      <inertial>
+        <origin xyz="0 0 0" rpy="0 0 0"/>
+        <mass value="0.0"/>
+        <inertia ixx="0" ixy="0" ixz="0" iyy="0" iyz="0" izz="0"/>
+      </inertial>
+      <xacro:common_link_visual
+        mesh_filename="lite6/visual/mounting"
+        origin_xyz="0 0 0"
+        origin_rpy="0 0 0"
+        material_name="${prefix}White" />
+      <xacro:common_link_collision
+        mesh_filename="lite6/collision/mounting"
+        origin_xyz="0 0 0"
+        origin_rpy="0 0 0" />
+    </link>
+    <!-- <joint name="realsense_joint" type="fixed"> -->
+    <!--   <parent link="mounting" /> -->
+    <!--   <child link = "camera_bottom_screw_frame" /> -->
+    <!--   <origin xyz="" rpy="0.0 0.0 0.0" /> -->
+    <!-- </joint> -->
+    <!-- camera urdf -->
+    <xacro:arg name="use_nominal_extrinsics" default="false"/>
+    <xacro:include filename="$(find realsense2_description)/urdf/_d405.urdf.xacro" />
+    <xacro:sensor_d405 parent="mounting" use_nominal_extrinsics="$(arg use_nominal_extrinsics)">
+      <origin xyz="-0.0005 0.0 0.007" rpy="0 0 0"/>
+    </xacro:sensor_d405>
   </xacro:macro>
 </robot>

Commit message: fix

File: xarm_description/urdf/lite6/lite6.urdf.xacro (robot description, xacro)
@@ -210,5 +210,5 @@
     <link name="${prefix}link_end" />
     <joint name="${prefix}joint_end" type="fixed">
-      <origin xyz="0 0 0.003" rpy="${pi} 0 ${pi/2}" />
+      <origin xyz="0 0 0.00" rpy="${pi} 0 ${pi/2}" />
       <parent link="${prefix}link6" />
       <child link="${prefix}link_end" />

Commit message: add xacro for rs415

File: xarm_description/urdf/lite6/lite6.urdf.xacro (robot description, xacro)
@@ -251,8 +251,39 @@
     <origin xyz="0.0 0.0 0.0625" rpy="0.0 0.0 0.0" />
     </joint>
+    <!-- camera 405 -->
+    <!-- <joint name="camera_mounting" type="fixed"> -->
+    <!-- <parent link="ft_sensor0_mech3"/> -->
+    <!-- <child link = "mounting" /> -->
+    <!--   <origin xyz="0.0 0.0 0.0" rpy="0.0 0.0 ${pi/2}"/> -->
+    <!-- </joint> -->
+    <!---->
+    <!-- <link name="mounting"> -->
+    <!--   <inertial> -->
+    <!--     <origin xyz="0 0 0" rpy="0 0 0"/> -->
+    <!--     <mass value="0.0"/> -->
+    <!--     <inertia ixx="0" ixy="0" ixz="0" iyy="0" iyz="0" izz="0"/> -->
+    <!--   </inertial> -->
+    <!--   <xacro:common_link_visual  -->
+    <!--     mesh_filename="lite6/visual/mounting"   -->
+    <!--     origin_xyz="0 0 0"  -->
+    <!--     origin_rpy="0 0 0" -->
+    <!--     material_name="${prefix}White" /> -->
+    <!--   <xacro:common_link_collision  -->
+    <!--     mesh_filename="lite6/collision/mounting"   -->
+    <!--     origin_xyz="0 0 0"  -->
+    <!--     origin_rpy="0 0 0" /> -->
+    <!-- </link> -->
+    <!---->
+    <!-- <xacro:arg name="use_nominal_extrinsics" default="false"/> -->
+    <!-- <xacro:include filename="$(find realsense2_description)/urdf/_d405.urdf.xacro" /> -->
+    <!---->
+    <!-- <xacro:sensor_d405 parent="mounting" use_nominal_extrinsics="$(arg use_nominal_extrinsics)"> -->
+    <!--  <origin xyz="-0.0005 0.0 0.007" rpy="0 0 0"/> -->
+    <!-- </xacro:sensor_d405> -->
+    <!-- 415 camera -->
     <joint name="camera_mounting" type="fixed">
     <parent link="ft_sensor0_mech3"/>
     <child link = "mounting" />
-      <origin xyz="0.0 0.0 0.0" rpy="0.0 0.0 ${pi/2}"/>
+      <origin xyz="0.0 0.0 0.0" rpy="0.0 0.0 ${pi}"/>
     </joint>
     <link name="mounting">
@@ -263,24 +294,18 @@
       </inertial>
       <xacro:common_link_visual
-        mesh_filename="lite6/visual/mounting"
-        origin_xyz="0 0 0"
-        origin_rpy="0 0 0"
-        material_name="${prefix}White" />
-      <xacro:common_link_collision
-        mesh_filename="lite6/collision/mounting"
-        origin_xyz="0 0 0"
-        origin_rpy="0 0 0" />
-    </link>
-    <!-- <joint name="realsense_joint" type="fixed"> -->
-    <!--   <parent link="mounting" /> -->
-    <!--   <child link = "camera_bottom_screw_frame" /> -->
-    <!--   <origin xyz="" rpy="0.0 0.0 0.0" /> -->
-    <!-- </joint> -->
-    <!-- camera urdf -->
+        mesh_filename="lite6/visual/d415_holder"
+        origin_xyz="0 0 0"
+        origin_rpy="0 0 0"
+        material_name="${prefix}White" />
+      <xacro:common_link_collision
+        mesh_filename="lite6/collision/d415_holder"
+        origin_xyz="0 0 0"
+        origin_rpy="0 0 0" />
+    </link>
     <xacro:arg name="use_nominal_extrinsics" default="false"/>
-    <xacro:include filename="$(find realsense2_description)/urdf/_d405.urdf.xacro" />
-    <xacro:sensor_d405 parent="mounting" use_nominal_extrinsics="$(arg use_nominal_extrinsics)">
-      <origin xyz="-0.0005 0.0 0.007" rpy="0 0 0"/>
-    </xacro:sensor_d405>
+    <xacro:include filename="$(find realsense2_description)/urdf/_d415.urdf.xacro" />
+    <xacro:sensor_d415 parent="mounting" use_nominal_extrinsics="$(arg use_nominal_extrinsics)">
+      <origin xyz="0.0 -0.001 0.0105" rpy="0 0 -${pi /2}"/>
+    </xacro:sensor_d415>
   </xacro:macro>
 </robot>
