Commit message: working on pointcloud action primitives

File: xarm_description/urdf/lite6/lite6_d405_knife.urdf.xacro (robot description, xacro)
@@ -239,5 +239,4 @@
         <origin xyz="0.0 0.0 0.0" rpy="0.0 0.0 0.0" />
         </joint>
-<!--
       <link name="knife">
         <inertial>
@@ -251,11 +250,11 @@
             origin_rpy="0.0 0.0 0.0"
             material_name="${prefix}Silver" />
-        </link> -->
-        <!-- <joint name="knife_base" type="fixed">
+        </link>
+        <joint name="knife_base" type="fixed">
         <parent link="tool_holder" />
         <child link = "knife" />
         <origin xyz="0.0 0.06 0.03" rpy="${-pi/2} ${pi/12} ${-pi/2}" />
-        <origin xyz="0.0 0.03 0.06" rpy="0.0 0.0 0.0" />
-        </joint> -->
+        <!-- <origin xyz="0.0 0.03 0.06" rpy="0.0 0.0 0.0" /> -->
+        </joint>
       <link
         name="probe">
@@ -264,6 +263,5 @@
       <parent link="ft_sensor0_wrench" />
       <child link = "probe" />
-      <!-- <origin xyz="-0.005 0.12 0.05" rpy="0.0 0.0 ${3*pi/2.0}" /> -->
-      <origin xyz="-0.003 0.00 0.14" rpy="0.0 ${pi/4} ${3*pi/2.0}" />
+      <origin xyz="-0.005 0.12 0.05" rpy="0.0 0.0 ${3*pi/2.0}" />
       </joint>
     <joint name="camera_mounting" type="fixed">

File: xarm_description/urdf/lite6/lite6_d405_probe.urdf.xacro (robot description, xacro)
@@ -210,5 +210,5 @@
     <link name="${prefix}link_end" />
     <joint name="${prefix}joint_end" type="fixed">
-      <origin xyz="0 0 0" rpy="${pi} 0 0" />
+      <origin xyz="0 0 0.00" rpy="${pi} 0 ${pi/2}" />
       <parent link="${prefix}link6" />
       <child link="${prefix}link_end" />
@@ -220,55 +220,96 @@
     <parent link="${prefix}link_end"/>
     <child link = "ft_sensor0_mounting" />
-    <origin xyz="0.0 0.0 0.0" rpy="${pi} 0.0 0.0" />
-    </joint>
-    <link name="tool_holder">
-        <inertial>
-          <origin rpy="0 0 0" xyz="0 0 0"/>
-          <mass value="0.0"/>
-          <inertia ixx="0" ixy="0" ixz="0" iyy="0" iyz="0" izz="0"/>
-        </inertial>
-        <xacro:common_link_visual
-            mesh_filename="lite6/visual/tool_holder"
-            origin_xyz="0 0 0.0"
-            origin_rpy="0 0 0"
-            material_name="${prefix}Silver" />
-        </link>
-        <joint name="base_tool" type="fixed">
-        <parent link="ft_sensor0_wrench" />
-        <child link = "tool_holder" />
-        <origin xyz="0.0 0.0 0.0" rpy="0.0 0.0 0.0" />
-        </joint>
-<!--
-      <link name="knife">
-        <inertial>
-          <origin rpy="0 0 0" xyz="0 0 0"/>
-          <mass value="0.0"/>
-          <inertia ixx="0" ixy="0" ixz="0" iyy="0" iyz="0" izz="0"/>
-        </inertial>
-        <xacro:common_link_visual
-            mesh_filename="lite6/visual/knife"
-            origin_xyz="0 0 0.0"
-            origin_rpy="0.0 0.0 0.0"
-            material_name="${prefix}Silver" />
-        </link> -->
-        <!-- <joint name="knife_base" type="fixed">
-        <parent link="tool_holder" />
-        <child link = "knife" />
-        <origin xyz="0.0 0.06 0.03" rpy="${-pi/2} ${pi/12} ${-pi/2}" />
-        <origin xyz="0.0 0.03 0.06" rpy="0.0 0.0 0.0" />
-        </joint> -->
-      <link
-        name="probe">
-      </link>
-      <joint name="tip_tool" type="fixed">
-      <parent link="ft_sensor0_wrench" />
-      <child link = "probe" />
-      <!-- <origin xyz="-0.005 0.12 0.05" rpy="0.0 0.0 ${3*pi/2.0}" /> -->
-      <origin xyz="-0.003 0.00 0.14" rpy="0.0 ${pi/4} ${3*pi/2.0}" />
-      </joint>
+    <origin xyz="0.0 0.0 0.0" rpy="${pi} 0.0 ${pi/2}" />
+    </joint>
+    <link name="probe_base">
+    <inertial>
+      <origin rpy="0 0 0" xyz="0 0 0"/>
+       <mass value="0.0"/>
+       <inertia ixx="0" ixy="0" ixz="0" iyy="0" iyz="0" izz="0"/>
+    </inertial>
+    <xacro:common_link_visual
+        mesh_filename="lite6/visual/punta_robot"
+        origin_xyz="0 0 0.01"
+        origin_rpy="0 0 0"
+        material_name="${prefix}Silver" />
+    <xacro:common_link_collision
+        mesh_filename="lite6/collision/punta_robot"
+        origin_xyz="0 0 0.01"
+        origin_rpy="0 0 0" />
+    </link>
+    <joint name="base_tool" type="fixed">
+    <parent link="ft_sensor0_wrench" />
+    <child link = "probe_base" />
+    <origin xyz="0.0 0.0 0.0" rpy="0.0 0.0 0.0" />
+    </joint>
+    <link
+      name="probe">
+    </link>
+    <joint name="tip_tool" type="fixed">
+    <parent link="ft_sensor0_wrench" />
+    <child link = "probe" />
+    <origin xyz="0.0 0.0 0.0625" rpy="0.0 0.0 0.0" />
+    </joint>
+    <!-- camera 405 -->
+    <!-- <joint name="camera_mounting" type="fixed"> -->
+    <!-- <parent link="ft_sensor0_mech3"/> -->
+    <!-- <child link = "mounting" /> -->
+    <!--   <origin xyz="0.0 0.0 0.0" rpy="0.0 0.0 ${pi/2}"/> -->
+    <!-- </joint> -->
+    <!---->
+    <!-- <link name="mounting"> -->
+    <!--   <inertial> -->
+    <!--     <origin xyz="0 0 0" rpy="0 0 0"/> -->
+    <!--     <mass value="0.0"/> -->
+    <!--     <inertia ixx="0" ixy="0" ixz="0" iyy="0" iyz="0" izz="0"/> -->
+    <!--   </inertial> -->
+    <!--   <xacro:common_link_visual  -->
+    <!--     mesh_filename="lite6/visual/mounting"   -->
+    <!--     origin_xyz="0 0 0"  -->
+    <!--     origin_rpy="0 0 0" -->
+    <!--     material_name="${prefix}White" /> -->
+    <!--   <xacro:common_link_collision  -->
+    <!--     mesh_filename="lite6/collision/mounting"   -->
+    <!--     origin_xyz="0 0 0"  -->
+    <!--     origin_rpy="0 0 0" /> -->
+    <!-- </link> -->
+    <!---->
+    <!-- <xacro:arg name="use_nominal_extrinsics" default="false"/> -->
+    <!-- <xacro:include filename="$(find realsense2_description)/urdf/_d405.urdf.xacro" /> -->
+    <!---->
+    <!-- <xacro:sensor_d405 parent="mounting" use_nominal_extrinsics="$(arg use_nominal_extrinsics)"> -->
+    <!--  <origin xyz="-0.0005 0.0 0.007" rpy="0 0 0"/> -->
+    <!-- </xacro:sensor_d405> -->
     <joint name="camera_mounting" type="fixed">
+  <parent link="ft_sensor0_mech3"/>
+  <child link="mounting"/>
+  <origin xyz="0.0 0.0 0.0" rpy="0.0 0.0 ${pi/2}"/>
+</joint>
+<link name="mounting">
+  <inertial>
+    <origin xyz="0 0 0" rpy="0 0 0"/>
+    <mass value="0.0"/>
+    <inertia ixx="0" ixy="0" ixz="0" iyy="0" iyz="0" izz="0"/>
+  </inertial>
+  <xacro:common_link_visual
+    mesh_filename="lite6/visual/mounting"
+    origin_xyz="0 0 0"
+    origin_rpy="0 0 0"
+    material_name="${prefix}White" />
+  <xacro:common_link_collision
+    mesh_filename="lite6/collision/mounting"
+    origin_xyz="0 0 0"
+    origin_rpy="0 0 0" />
+</link>
+<xacro:arg name="use_nominal_extrinsics" default="false"/>
+<xacro:include filename="$(find realsense2_description)/urdf/_d405.urdf.xacro" />
+<xacro:sensor_d405 parent="mounting" use_nominal_extrinsics="$(arg use_nominal_extrinsics)">
+  <origin xyz="-0.0005 0.0 0.007" rpy="0 0 0"/>
+</xacro:sensor_d405>
+    <!-- 415 camera -->
+    <!-- <joint name="camera_mounting" type="fixed">
     <parent link="ft_sensor0_mech3"/>
     <child link = "mounting" />
-      <origin xyz="0.0 0.0 0.0" rpy="0.0 0.0 ${pi/2}"/>
+      <origin xyz="0.0 0.0 0.0" rpy="0.0 0.0 ${pi}"/>
     </joint>
     <link name="mounting">
@@ -276,21 +317,21 @@
         <origin xyz="0 0 0" rpy="0 0 0"/>
         <mass value="0.0"/>
-        <inertia ixx="0" ixy="0" ixz="0" iyy="0" iyz="0" izz="0"/>/
+        <inertia ixx="0" ixy="0" ixz="0" iyy="0" iyz="0" izz="0"/>
       </inertial>
       <xacro:common_link_visual
-        mesh_filename="lite6/visual/mounting"
-        origin_xyz="0 0 0"
-        origin_rpy="0 0 0"
-        material_name="${prefix}White" />
-      <!-- <xacro:common_link_collision
-        mesh_filename="lite6/collision/mounting"
-        origin_xyz="0 0 0"
-        origin_rpy="0 0 0" /> -->
+        mesh_filename="lite6/visual/d415_holder"
+        origin_xyz="0 0 0"
+        origin_rpy="0 0 0"
+        material_name="${prefix}White" />
+      <xacro:common_link_collision
+        mesh_filename="lite6/collision/d415_holder"
+        origin_xyz="0 0 0"
+        origin_rpy="0 0 0" />
     </link>
     <xacro:arg name="use_nominal_extrinsics" default="false"/>
-    <xacro:include filename="$(find realsense2_description)/urdf/_d405.urdf.xacro" />
-    <xacro:sensor_d405 parent="mounting" use_nominal_extrinsics="$(arg use_nominal_extrinsics)">
-      <origin xyz="-0.0005 0.0 0.007" rpy="0 0 0"/>
-    </xacro:sensor_d405>
+    <xacro:include filename="$(find realsense2_description)/urdf/_d415.urdf.xacro" />
+    <xacro:sensor_d415 parent="mounting" use_nominal_extrinsics="$(arg use_nominal_extrinsics)">
+      <origin xyz="0.0 -0.001 0.0105" rpy="0 0 -${pi /2}"/>
+    </xacro:sensor_d415> -->
   </xacro:macro>
 </robot>
