Commit message: peeling experiments

File: xarm_description/urdf/lite6/lite6_d405_peeler.urdf.xacro (robot description, xacro)
@@ -265,6 +265,5 @@
       <child link = "probe" />
       <!-- <origin xyz="-0.005 0.12 0.05" rpy="0.0 0.0 ${3*pi/2.0}" /> -->
-      <!-- <origin xyz="-0.005 0.00 0.12" rpy="0.0 ${pi/4} ${3*pi/2.0}" /> -->
-      <origin xyz="-0.005 0.07 0.015" rpy="0.0 0.0 0.0" />
+      <origin xyz="-0.005 0.00 0.12" rpy="0.0 ${pi/4} ${3*pi/2.0}" />
       </joint>
     <joint name="camera_mounting" type="fixed">
