Commit message: Fix peeler knife orientation in D405 peeler URDF
Correct tip_tool joint rpy from pi/2 to -pi/2 for proper knife alignment.

Co-Authored-By: Claude Opus 4.6 <noreply@anthropic.com>

File: xarm_description/urdf/lite6/lite6_d405_peeler.urdf.xacro (robot description, xacro)
@@ -264,5 +264,5 @@
     <parent link="tool_holder" />
     <child link = "peeler" />
-    <origin xyz="0.0 0.0 0.02" rpy="${pi} 0.0 ${pi/2}" />
+    <origin xyz="0.0 0.0 0.02" rpy="${pi} 0.0 ${-pi/2}" />
     </joint>
     <!-- Probe frame at the tip of the knife -->

Commit message: Flip probe frame z-axis and update RViz config
Rotate probe joint by pi around x-axis so z+ points toward the
object surface. Update RViz display config.

Co-Authored-By: Claude Opus 4.6 <noreply@anthropic.com>

File: xarm_description/urdf/lite6/lite6_d405_peeler.urdf.xacro (robot description, xacro)
@@ -271,5 +271,5 @@
     <parent link="peeler" />
     <child link = "probe" />
-    <origin xyz="-0.05 0.0 0.0" rpy="0.0 0.0 ${-pi/2}" />
+    <origin xyz="-0.05 0.0 0.0" rpy="${pi} 0.0 ${-pi/2}" />
     </joint>
     <!-- D405 camera with mounting holder -->
