Commit message: Add custom tool chain, compliance controller, and SRDF fixes for lite6
- lite6.urdf.xacro: Add Bota FT sensor, camera mount, RealSense D415,
  and probe tip to lite6 kinematic chain with collision/visual meshes
- lite6_controllers.yaml: Add cartesian_compliance_controller config
  with Bota FT sensor integration, tune stiffness/PD gains for safe
  teleop; increase controller_manager update rate to 250 Hz;
  set end_effector_link to "probe" for all cartesian controllers
- _lite6_macro.srdf.xacro: Extend planning group chain through FT sensor
  to probe tip; add disable_collisions entries for custom tool links
  (FT sensor, camera mount, camera, probe) to fix MoveIt planning
- _ros2_control.launch.py: Add cartesian controller spawners (inactive)
- display.rviz: Add wrench and F/T sensor visualization
- Add STL meshes for d415_holder, mounting, punta_robot, punta_ur_5mm

Co-Authored-By: Claude Opus 4.6 <noreply@anthropic.com>

File: xarm_description/urdf/lite6/lite6_original.urdf.xacro (robot description, xacro)
@@ -208,104 +208,10 @@
       <dynamics damping="1.0" friction="1.0"/>
     </joint>
-    <link name="${prefix}link_end" />
-    <joint name="${prefix}joint_end" type="fixed">
-      <origin xyz="0 0 0.00" rpy="${pi} 0 ${pi/2}" />
+    <!-- <link name="${prefix}link_eef" />
+    <joint name="${prefix}joint_eef" type="fixed">
+      <origin xyz="0 0 0" rpy="0 0 0" />
       <parent link="${prefix}link6" />
-      <child link="${prefix}link_end" />
-    </joint>
-    <!-- force sensor urdf -->
-    <xacro:include filename="$(find bota_driver)/urdf/BFT_SENS_ECAT_M8.urdf.xacro" />
-    <xacro:BFT_SENS_ECAT_M8 prefix="ft_sensor0" />
-    <joint name="bota_ft_sensor" type="fixed">
-    <parent link="${prefix}link_end"/>
-    <child link = "ft_sensor0_mounting" />
-    <origin xyz="0.0 0.0 0.0" rpy="${pi} 0.0 ${pi/2}" />
-    </joint>
-    <link name="probe_base">
-    <inertial>
-      <origin rpy="0 0 0" xyz="0 0 0"/>
-       <mass value="0.0"/>
-       <inertia ixx="0" ixy="0" ixz="0" iyy="0" iyz="0" izz="0"/>
-    </inertial>
-    <xacro:common_link_visual
-        mesh_filename="lite6/visual/punta_robot"
-        origin_xyz="0 0 0.01"
-        origin_rpy="0 0 0"
-        material_name="${prefix}Silver" />
-    <xacro:common_link_collision
-        mesh_filename="lite6/collision/punta_robot"
-        origin_xyz="0 0 0.01"
-        origin_rpy="0 0 0" />
-    </link>
-    <joint name="base_tool" type="fixed">
-    <parent link="ft_sensor0_wrench" />
-    <child link = "probe_base" />
-    <origin xyz="0.0 0.0 0.0" rpy="0.0 0.0 0.0" />
-    </joint>
-    <link
-      name="probe">
-    </link>
-    <joint name="tip_tool" type="fixed">
-    <parent link="ft_sensor0_wrench" />
-    <child link = "probe" />
-    <origin xyz="0.0 0.0 0.0625" rpy="0.0 0.0 0.0" />
-    </joint>
-    <!-- camera 405 -->
-    <!-- <joint name="camera_mounting" type="fixed"> -->
-    <!-- <parent link="ft_sensor0_mech3"/> -->
-    <!-- <child link = "mounting" /> -->
-    <!--   <origin xyz="0.0 0.0 0.0" rpy="0.0 0.0 ${pi/2}"/> -->
-    <!-- </joint> -->
-    <!---->
-    <!-- <link name="mounting"> -->
-    <!--   <inertial> -->
-    <!--     <origin xyz="0 0 0" rpy="0 0 0"/> -->
-    <!--     <mass value="0.0"/> -->
-    <!--     <inertia ixx="0" ixy="0" ixz="0" iyy="0" iyz="0" izz="0"/> -->
-    <!--   </inertial> -->
-    <!--   <xacro:common_link_visual  -->
-    <!--     mesh_filename="lite6/visual/mounting"   -->
-    <!--     origin_xyz="0 0 0"  -->
-    <!--     origin_rpy="0 0 0" -->
-    <!--     material_name="${prefix}White" /> -->
-    <!--   <xacro:common_link_collision  -->
-    <!--     mesh_filename="lite6/collision/mounting"   -->
-    <!--     origin_xyz="0 0 0"  -->
-    <!--     origin_rpy="0 0 0" /> -->
-    <!-- </link> -->
-    <!---->
-    <!-- <xacro:arg name="use_nominal_extrinsics" default="false"/> -->
-    <!-- <xacro:include filename="$(find realsense2_description)/urdf/_d405.urdf.xacro" /> -->
-    <!---->
-    <!-- <xacro:sensor_d405 parent="mounting" use_nominal_extrinsics="$(arg use_nominal_extrinsics)"> -->
-    <!--  <origin xyz="-0.0005 0.0 0.007" rpy="0 0 0"/> -->
-    <!-- </xacro:sensor_d405> -->
-    <!-- 415 camera -->
-    <joint name="camera_mounting" type="fixed">
-    <parent link="ft_sensor0_mech3"/>
-    <child link = "mounting" />
-      <origin xyz="0.0 0.0 0.0" rpy="0.0 0.0 ${pi}"/>
-    </joint>
-    <link name="mounting">
-      <inertial>
-        <origin xyz="0 0 0" rpy="0 0 0"/>
-        <mass value="0.0"/>
-        <inertia ixx="0" ixy="0" ixz="0" iyy="0" iyz="0" izz="0"/>
-      </inertial>
-      <xacro:common_link_visual
-        mesh_filename="lite6/visual/d415_holder"
-        origin_xyz="0 0 0"
-        origin_rpy="0 0 0"
-        material_name="${prefix}White" />
-      <xacro:common_link_collision
-        mesh_filename="lite6/collision/d415_holder"
-        origin_xyz="0 0 0"
-        origin_rpy="0 0 0" />
-    </link>
-    <xacro:arg name="use_nominal_extrinsics" default="false"/>
-    <xacro:include filename="$(find realsense2_description)/urdf/_d415.urdf.xacro" />
-    <xacro:sensor_d415 parent="mounting" use_nominal_extrinsics="$(arg use_nominal_extrinsics)">
-      <origin xyz="0.0 -0.001 0.0105" rpy="0 0 -${pi /2}"/>
-    </xacro:sensor_d415>
+      <child link="${prefix}link_eef" />
+    </joint> -->
   </xacro:macro>
 </robot>

File: xarm_moveit_config/srdf/_lite6_macro.srdf.xacro (robot description, xacro)
@@ -19,5 +19,9 @@
       <joint name="${prefix}joint5" />
       <joint name="${prefix}joint6" />
-      <joint name="${prefix}joint_eef" />
+      <!-- Extend to probe tip via FT sensor chain (link6 → link_end → ft_sensor0 → probe) -->
+      <joint name="${prefix}joint_end" />
+      <joint name="bota_ft_sensor" />
+      <joint name="ft_sensor0_mounting_to_wrench" />
+      <joint name="tip_tool" />
       <!-- To count in gripper TCP offset, if no need, please uncomment following 2 lines -->
       <xacro:if value="${add_gripper}">
@@ -95,4 +99,20 @@
     <disable_collisions link1="${prefix}link5" link2="${prefix}link_eef" reason="Never" />
     <disable_collisions link1="${prefix}link6" link2="${prefix}link_eef" reason="Adjacent" />
+    <!-- Custom tool chain: FT sensor, camera mount, camera, probe (bota + realsense) -->
+    <disable_collisions link1="${prefix}link6" link2="ft_sensor0_mounting" reason="Never" />
+    <disable_collisions link1="${prefix}link6" link2="mounting" reason="Never" />
+    <disable_collisions link1="${prefix}link6" link2="probe_base" reason="Never" />
+    <disable_collisions link1="${prefix}link_eef" link2="ft_sensor0_mounting" reason="Never" />
+    <disable_collisions link1="${prefix}link_eef" link2="mounting" reason="Never" />
+    <disable_collisions link1="${prefix}link_eef" link2="camera_link" reason="Never" />
+    <disable_collisions link1="${prefix}link5" link2="ft_sensor0_mounting" reason="Never" />
+    <disable_collisions link1="${prefix}link5" link2="mounting" reason="Never" />
+    <disable_collisions link1="ft_sensor0_mounting" link2="mounting" reason="Never" />
+    <disable_collisions link1="ft_sensor0_mounting" link2="camera_link" reason="Never" />
+    <disable_collisions link1="ft_sensor0_mounting" link2="probe_base" reason="Never" />
+    <disable_collisions link1="mounting" link2="camera_link" reason="Adjacent" />
+    <disable_collisions link1="mounting" link2="probe_base" reason="Never" />
+    <disable_collisions link1="${prefix}link_end" link2="ft_sensor0_mounting" reason="Adjacent" />
+    <disable_collisions link1="${prefix}link_end" link2="probe_base" reason="Never" />
   </xacro:macro>
 </robot>
